File: Kyamaries-HPS-Clock.kicad_pcb (KiCad board)
At the start: 2 copper layers, 140 x 90 mm, 59 parts, among them J1 Conn_01x06, J2 Power_inlet_vertical, J3 Conn_02x03_Odd_Even, SW1 Omron_B3F_SPST, SW2 Omron_B3F_SPST, SW3 Omron_B3F_SPST, SW4 Omron_B3F_SPST, SW5 Omron_B3F_SPST, U1 ATmega328-PU, U2 L7805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

Commit message: Updated schematics
Routing:
- net GND: track 545.7 -> 504.6 mm, vias 17 -> 20
- net Net-(C2-Pad1): track 28.5 -> 32.1 mm
Changed lines of the file:
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@@
     (fp_arc (start -0.29972 8.49884) (mid -0.153162 8.145018) (end 0.20066 7.99846) (layer "F.SilkS") (width 0.12))
     (fp_arc (start 0.20066 22.9997) (mid -0.153162 22.853142) (end -0.29972 22.49932) (layer "F.SilkS") (width 0.12))
-    (fp_arc (start 64.20104 22.49932) (mid 64.054482 22.853142) (end 63.70066 22.9997) (layer "F.SilkS") (width 0.12))
+    (fp_arc (start 64.20104 22.49932) (mid 64.054473 22.853115) (end 63.70066 22.9997) (layer "F.SilkS") (width 0.12))
     (fp_line (start 72.25 -2.75) (end 72.25 33.75) (layer "F.CrtYd") (width 0.05))
     (fp_line (start -8.25 33.75) (end 72.25 33.75) (layer "F.CrtYd") (width 0.05))
@@
     (effects (font (size 2 2) (thickness 0.15)))
   )
-  (gr_text "{dblquote}The Beginning{dblquote}" (at 104.14 137.16) (layer "F.SilkS")
-    (effects (font (size 2 2) (thickness 0.15)))
+  (gr_text "{dblquote}The Beginning{dblquote}" (at 105.029671 132.151854) (layer "F.SilkS")
+    (effects (font (size 2.5 2.5) (thickness 0.15)))
   )
   (gr_text "SELECT" (at 203.2 101.6) (layer "F.SilkS")
@@
   (segment (start 107.936314 119.379984) (end 107.936314 107.963686) (width 0.2032) (layer "F.Cu") (net 2))
   (segment (start 143.208845 136.888074) (end 143.208845 132.581359) (width 0.2032) (layer "F.Cu") (net 2))
-  (segment (start 101.82 95.18) (end 101.113952 95.886048) (width 0.2032) (layer "F.Cu") (net 2))
   (segment (start 131.1682 134.62) (end 130.39 134.62) (width 0.2032) (layer "F.Cu") (net 2))
   (segment (start 158.5 67.06) (end 158.901109 67.06) (width 0.2032) (layer "F.Cu") (net 2))
@@
   (segment (start 197.83 66.33) (end 198.982009 66.33) (width 0.2032) (layer "F.Cu") (net 2))
   (segment (start 159.18963 58.383184) (end 160.88963 58.383184) (width 0.2032) (layer "F.Cu") (net 2))
-  (segment (start 109.889138 80.422533) (end 109.889138 78.516805) (width 0.2032) (layer "F.Cu") (net 2))
   (segment (start 145.483074 136.888074) (end 143.208845 136.888074) (width 0.2032) (layer "F.Cu") (net 2))
   (segment (start 120.622694 115.563719) (end 122.086582 115.563719) (width 0.2032) (layer "F.Cu") (net 2))
+  (segment (start 91.44 83.82) (end 91.44 78.74) (width 2) (layer "F.Cu") (net 2))
   (segment (start 155.765998 141.540207) (end 155.79 141.516205) (width 0.2032) (layer "F.Cu") (net 2))
   (segment (start 107.53 107.557372) (end 107.53 96.52) (width 0.2032) (layer "F.Cu") (net 2))
@@
   (segment (start 122.086582 115.563719) (end 122.810735 114.839566) (width 0.2032) (layer "F.Cu") (net 2))
   (segment (start 195.58 107.949494) (end 196.448826 107.080668) (width 0.2032) (layer "F.Cu") (net 2))
-  (segment (start 95.730003 95.886048) (end 91.44 91.596045) (width 0.2032) (layer "F.Cu") (net 2))
   (segment (start 150.325078 124.865818) (end 150.529022 124.661874) (width 0.2032) (layer "F.Cu") (net 2))
   (segment (start 146.06 132.199583) (end 146.06 130.8) (width 0.2032) (layer "F.Cu") (net 2))
@@
   (segment (start 105.83 79.924152) (end 105.83 78.74) (width 0.2032) (layer "F.Cu") (net 2))
   (segment (start 179.7621 133.246873) (end 183.37512 129.633853) (width 0.2032) (layer "F.Cu") (net 2))
-  (segment (start 91.44 78.74) (end 91.44 91.9) (width 0.5) (layer "F.Cu") (net 2))
   (segment (start 145.205818 124.865818) (end 143.52 123.18) (width 0.2032) (layer "F.Cu") (net 2))
   (segment (start 132.599629 112.66935) (end 132.740623 112.528356) (width 0.2032) (layer "F.Cu") (net 2))
@@
   (segment (start 199.2 74.74) (end 198.12 73.66) (width 0.2032) (layer "F.Cu") (net 2))
   (segment (start 195.58 114.3) (end 198.095689 116.815689) (width 0.2032) (layer "F.Cu") (net 2))
+  (segment (start 86.36 78.74) (end 91.44 78.74) (width 2) (layer "F.Cu") (net 2))
   (segment (start 135.442578 129.695689) (end 134.62 130.518267) (width 0.2032) (layer "F.Cu") (net 2))
   (segment (start 134.1641 132.5616) (end 134.1641 131.6241) (width 0.2032) (layer "F.Cu") (net 2))
@@
   (segment (start 199.2 79.03) (end 199.2 74.74) (width 0.2032) (layer "F.Cu") (net 2))
   (segment (start 200.66 123.19) (end 198.095689 120.625689) (width 0.2032) (layer "F.Cu") (net 2))
-  (segment (start 101.6 68.58) (end 91.44 78.74) (width 0.2032) (layer "F.Cu") (net 2))
   (segment (start 193.854727 133.246873) (end 198.02718 137.419326) (width 0.2032) (layer "F.Cu") (net 2))
   (segment (start 150.529022 124.661874) (end 150.730896 124.46) (width 0.2032) (layer "F.Cu") (net 2))
@@
   (segment (start 195.58 68.58) (end 197.83 66.33) (width 0.2032) (layer "F.Cu") (net 2))
   (segment (start 149.232432 141.540207) (end 155.765998 141.540207) (width 0.2032) (layer "F.Cu") (net 2))
-  (segment (start 109.889138 78.516805) (end 120.112972 68.292971) (width 0.2032) (layer "F.Cu") (net 2))
   (segment (start 143.52 123.18) (end 137.004311 129.695689) (width 0.2032) (layer "F.Cu") (net 2))
   (segment (start 148.17 139.7) (end 148.17 140.477775) (width 0.2032) (layer "F.Cu") (net 2))
@@
   (segment (start 154.94 114.3) (end 154.94 123.481733) (width 0.2032) (layer "F.Cu") (net 2))
   (segment (start 132.740623 112.528356) (end 132.740623 110.516279) (width 0.2032) (layer "F.Cu") (net 2))
+  (segment (start 91.44 73.66) (end 91.44 78.74) (width 2) (layer "F.Cu") (net 2))
   (segment (start 178.403232 133.246873) (end 179.7621 133.246873) (width 0.2032) (layer "F.Cu") (net 2))
   (segment (start 142.415689 124.284311) (end 143.52 123.18) (width 0.2032) (layer "F.Cu") (net 2))
@@
   (segment (start 143.502818 132.287386) (end 145.869307 132.287386) (width 0.2032) (layer "F.Cu") (net 2))
   (segment (start 148.17 139.575) (end 145.483074 136.888074) (width 0.2032) (layer "F.Cu") (net 2))
-  (segment (start 101.113952 95.886048) (end 95.730003 95.886048) (width 0.2032) (layer "F.Cu") (net 2))
   (segment (start 107.53 82.781671) (end 109.889138 80.422533) (width 0.2032) (layer "F.Cu") (net 2))
+  (via (at 91.44 73.66) (size 0.8128) (drill 0.4064) (layers "F.Cu" "B.Cu") (net 2))
   (via (at 195.58 114.3) (size 0.8128) (drill 0.4064) (layers "F.Cu" "B.Cu") (net 2))
   (via (at 198.12 73.66) (size 0.8128) (drill 0.4064) (layers "F.Cu" "B.Cu") (net 2))
   (via (at 132.599629 112.66935) (size 0.8128) (drill 0.4064) (layers "F.Cu" "B.Cu") (net 2))
+  (via (at 86.36 78.74) (size 0.8128) (drill 0.4064) (layers "F.Cu" "B.Cu") (net 2))
   (via (at 109.889138 80.422533) (size 0.8128) (drill 0.4064) (layers "F.Cu" "B.Cu") (net 2))
   (via (at 145.205818 124.865818) (size 0.8128) (drill 0.4064) (layers "F.Cu" "B.Cu") (net 2))
@@
   (via (at 122.810735 114.839566) (size 0.8128) (drill 0.4064) (layers "F.Cu" "B.Cu") (net 2))
   (via (at 157.48 66.04) (size 0.8128) (drill 0.4064) (layers "F.Cu" "B.Cu") (net 2))
+  (via (at 91.44 83.82) (size 0.8128) (drill 0.4064) (layers "F.Cu" "B.Cu") (net 2))
   (via (at 106.68 86.36) (size 0.8128) (drill 0.4064) (layers "F.Cu" "B.Cu") (net 2))
   (via (at 201.930129 137.849166) (size 0.8128) (drill 0.4064) (layers "F.Cu" "B.Cu") (net 2))
@@
   (segment (start 145.205818 124.865818) (end 148.495092 124.865818) (width 0.2032) (layer "B.Cu") (net 2))
   (segment (start 197.36382 106.165674) (end 197.36382 93.245531) (width 0.2032) (layer "B.Cu") (net 2))
-  (segment (start 97.95 81.02) (end 105.83 88.9) (width 0.2032) (layer "F.Cu") (net 3))
-  (segment (start 96.52432 97.48432) (end 104.86568 97.48432) (width 0.2032) (layer "F.Cu") (net 3))
-  (segment (start 105.83 96.52) (end 105.83 88.9) (width 0.2032) (layer "F.Cu") (net 3))
-  (segment (start 104.86568 97.48432) (end 105.83 96.52) (width 0.2032) (layer "F.Cu") (net 3))
-  (segment (start 96.52 97.48) (end 96.52432 97.48432) (width 0.2032) (layer "F.Cu") (net 3))
+  (segment (start 105.62 88.9) (end 97.74 81.02) (width 1.5) (layer "F.Cu") (net 3))
+  (segment (start 105.752289 99.392618) (end 105.752289 96.52) (width 2) (layer "F.Cu") (net 3))
+  (segment (start 105.83 88.9) (end 105.83 96.52) (width 1.5) (layer "F.Cu") (net 3))
+  (segment (start 105.466514 99.678393) (end 105.752289 99.392618) (width 2) (layer "F.Cu") (net 3))
+  (segment (start 96.52 97.48) (end 98.943275 97.48) (width 2) (layer "F.Cu") (net 3))
+  (segment (start 101.141668 99.678393) (end 105.466514 99.678393) (width 2) (layer "F.Cu") (net 3))
+  (segment (start 105.83 88.9) (end 105.62 88.9) (width 1.5) (layer "F.Cu") (net 3))
+  (segment (start 98.943275 97.48) (end 101.141668 99.678393) (width 2) (layer "F.Cu") (net 3))
   (segment (start 204.89 134.62) (end 201.93 134.62) (width 0.2032) (layer "F.Cu") (net 4))
   (segment (start 201.93 134.62) (end 200.66 133.35) (width 0.2032) (layer "F.Cu") (net 4))
